Commit message: Updating urdf

File: cambot_description/urdf/cambot.urdf (robot description, URDF)
Before this commit: robot cambot, 4 links, 3 joints
Links:
- removed link servo_link
- link camera_link: geometry visual mesh filename=package://cambot_description/meshes/camera_conjunt.stl
Joints:
- removed joint base_to_servo
- removed joint servo_to_camera
- added joint base_to_camera: type continuous, parent base_link, child camera_link, origin xyz=0.3 -0.15 0.5 rpy=-1.57 0 0, axis 0 0 1
- joint cambot_world: axis (none) -> 0 0 1; origin xyz=0 0 0 rpy=-1.57 -1.57 0 -> xyz=0 0 0.5 rpy=0 0 0

Commit message: Updating urdf

File: cambot_description/urdf/cambot.urdf (robot description, URDF)
Before this commit: robot cambot, 3 links, 2 joints
Links:
- removed link world
- added link base_footprint
- added link camera_support_link; visual mesh filename=package://cambot_description/meshes/cambot_camera_support.s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
- added link left_wheel_link; visual mesh filename=package://cambot_description/meshes/cambot_wheel.stl
- added link right_wheel_link; visual mesh filename=package://cambot_description/meshes/cambot_wheel.stl
- added link servo_link; visual mesh filename=package://cambot_description/meshes/cambot_servo.stl
- link base_link: geometry visual mesh filename=package://cambot_description/meshes/cambot_base.stl
- link camera_link: geometry visual mesh filename=package://cambot_description/meshes/cambot_camera.stl
Joints:
- removed joint base_to_camera
- removed joint cambot_world
- added joint base_footprint_joint: type fixed, parent base_footprint, child base_link, origin xyz=0 0 0 rpy=0 0 0
- added joint base_to_left_wheel: type continuous, parent base_link, child left_wheel_link, origin xyz=0.21 0.50 0.28 rpy=-1.57 0 0, axis 0 0 1
- added joint base_to_right_wheel: type continuous, parent base_link, child right_wheel_link, origin xyz=0.21 -0.50 0.28 rpy=1.57 0 0, axis 0 0 1
- added joint base_to_servo: type fixed, parent base_link, child servo_link, origin xyz=0.2 -0.21 1.035 rpy=-1.57 0 0
- added joint camera_support_to_camera: type fixed, parent camera_support_link, child camera_link, origin xyz=0.2 -0.35 0.35 rpy=1.57 0 0
- added joint servo_to_camera_support: type revolute, parent servo_link, child camera_support_link, origin xyz=0 0 0 rpy=0 0 0, axis 0 0 1, limit lower=-0.4 upper=0.4 effort=10.0 velocity=0.5
