Commit message: Updating cambot_control

File: cambot_control/cambot_description/urdf/cambot.urdf (robot description, URDF)
Before this commit: robot cambot, 7 links, 6 joints
Links:
- link camera_support_link: mass None -> 0.051725
- link left_wheel_link: mass None -> 0.01311625
- link right_wheel_link: mass None -> 0.01311625
- link servo_link: mass None -> 0.056861
